Commit message: refactor: replace hardcoded rotation values with pi-based expressions in robot URDF files

File: src/gizmo/gizmo_description/urdf/include/base_floor1.xacro (robot description, xacro)
@@ -17,5 +17,5 @@
         <!-- Part bn_8699_1727796_hexagon_socket_button_head_screw_m2_5x6 -->
         <visual>
-        <origin xyz="0.0217 0.0627386 0.00961" rpy="3.14159 0 -1.5708"/>
+        <origin xyz="0.0217 0.0627386 0.00961" rpy="${pi} 0 -${pi/2}"/>
         <geometry>
             <mesh filename="package://gizmo_description/meshes/bn_8699_1727796_hexagon_socket_button_head_screw_m2_5x6.stl"/>
@@ -27,5 +27,5 @@
         <!-- Part standoff_spacer_m3_30mm -->
         <visual>
-        <origin xyz="-0.0444488 -0.0371773 0.0035" rpy="0 -0 0"/>
+        <origin xyz="-0.0444488 -0.0371773 0.0035" rpy="0 0 0"/>
         <geometry>
             <mesh filename="package://gizmo_description/meshes/standoff_spacer_m3_30mm.stl"/>
@@ -37,5 +37,5 @@
         <!-- Part bn_1593_1348663_hexagon_socket_button_head_screw_m3x6 -->
         <visual>
-        <origin xyz="-0.0444488 -0.0371773 0.001" rpy="-0 -1.5708 0"/>
+        <origin xyz="-0.0444488 -0.0371773 0.001" rpy="0 -${pi/2} 0"/>
         <geometry>
             <mesh filename="package://gizmo_description/meshes/bn_1593_1348663_hexagon_socket_button_head_screw_m3x6.stl"/>
@@ -47,5 +47,5 @@
         <!-- Part bn_8699_1727796_hexagon_socket_button_head_screw_m2_5x6_2 -->
         <visual>
-        <origin xyz="0.001 -0.0627386 0.00961" rpy="1.5708 -0 1.5708"/>
+        <origin xyz="0.001 -0.0627386 0.00961" rpy="${pi/2} 0 ${pi/2}"/>
         <geometry>
             <mesh filename="package://gizmo_description/meshes/bn_8699_1727796_hexagon_socket_button_head_screw_m2_5x6.stl"/>
@@ -57,5 +57,5 @@
         <!-- Part standoff_spacer_m3_30mm_2 -->
         <visual>
-        <origin xyz="-0.0444488 0.0371773 0.0035" rpy="0 -0 0"/>
+        <origin xyz="-0.0444488 0.0371773 0.0035" rpy="0 0 0"/>
         <geometry>
             <mesh filename="package://gizmo_description/meshes/standoff_spacer_m3_30mm.stl"/>
@@ -67,5 +67,5 @@
         <!-- Part bn_1593_1348663_hexagon_socket_button_head_screw_m3x6_2 -->
         <visual>
-        <origin xyz="-0.00011 -0.0337386 0.001" rpy="-0 -1.5708 0"/>
+        <origin xyz="-0.00011 -0.0337386 0.001" rpy="0 -${pi/2} 0"/>
         <geometry>
             <mesh filename="package://gizmo_description/meshes/bn_1593_1348663_hexagon_socket_button_head_screw_m3x6.stl"/>
@@ -77,5 +77,5 @@
         <!-- Part bn_1593_1348663_hexagon_socket_button_head_screw_m3x6_3 -->
         <visual>
-        <origin xyz="-0.00011 0.0337386 0.001" rpy="-0 -1.5708 0"/>
+        <origin xyz="-0.00011 0.0337386 0.001" rpy="0 -${pi/2} 0"/>
         <geometry>
             <mesh filename="package://gizmo_description/meshes/bn_1593_1348663_hexagon_socket_button_head_screw_m3x6.stl"/>
@@ -87,5 +87,5 @@
         <!-- Part bn_8699_1727796_hexagon_socket_button_head_screw_m2_5x6_3 -->
         <visual>
-        <origin xyz="0.0217 -0.0627386 0.00961" rpy="1.5708 -0 1.5708"/>
+        <origin xyz="0.0217 -0.0627386 0.00961" rpy="${pi/2} 0 ${pi/2}"/>
         <geometry>
             <mesh filename="package://gizmo_description/meshes/bn_8699_1727796_hexagon_socket_button_head_screw_m2_5x6.stl"/>
@@ -97,5 +97,5 @@
         <!-- Part bn_1593_1348663_hexagon_socket_button_head_screw_m3x6_4 -->
         <visual>
-        <origin xyz="0.03511 0.0557386 0.001" rpy="-0 -1.5708 0"/>
+        <origin xyz="0.03511 0.0557386 0.001" rpy="0 -${pi/2} 0"/>
         <geometry>
             <mesh filename="package://gizmo_description/meshes/bn_1593_1348663_hexagon_socket_button_head_screw_m3x6.stl"/>
@@ -107,5 +107,5 @@
         <!-- Part base_floor_1 -->
         <visual>
-        <origin xyz="0 0 0" rpy="0 -0 0"/>
+        <origin xyz="0 0 0" rpy="0 0 0"/>
         <geometry>
             <mesh filename="package://gizmo_description/meshes/base_floor_1.stl"/>
@@ -117,5 +117,5 @@
         <!-- Part servo_bracket_r -->
         <visual>
-        <origin xyz="0.0175 -0.0447386 0.0035" rpy="0 -0 0"/>
+        <origin xyz="0.0175 -0.0447386 0.0035" rpy="0 0 0"/>
         <geometry>
             <mesh filename="package://gizmo_description/meshes/servo_bracket_r.stl"/>
@@ -127,5 +127,5 @@
         <!-- Part bn_1593_1348663_hexagon_socket_button_head_screw_m3x6_5 -->
         <visual>
-        <origin xyz="0.03511 0.0337386 0.001" rpy="-0 -1.5708 0"/>
+        <origin xyz="0.03511 0.0337386 0.001" rpy="0 -${pi/2} 0"/>
         <geometry>
             <mesh filename="package://gizmo_description/meshes/bn_1593_1348663_hexagon_socket_button_head_screw_m3x6.stl"/>
@@ -137,5 +137,5 @@
         <!-- Part servo_bracket_l -->
         <visual>
-        <origin xyz="0.0175 0.0447386 0.0035" rpy="0 -0 0"/>
+        <origin xyz="0.0175 0.0447386 0.0035" rpy="0 0 0"/>
         <geometry>
             <mesh filename="package://gizmo_description/meshes/servo_bracket_l.stl"/>
@@ -147,5 +147,5 @@
         <!-- Part bn_1593_1348663_hexagon_socket_button_head_screw_m3x6_6 -->
         <visual>
-        <origin xyz="-0.0444488 0.0371773 0.001" rpy="-0 -1.5708 0"/>
+        <origin xyz="-0.0444488 0.0371773 0.001" rpy="0 -${pi/2} 0"/>
         <geometry>
             <mesh filename="package://gizmo_description/meshes/bn_1593_1348663_hexagon_socket_button_head_screw_m3x6.stl"/>
@@ -157,5 +157,5 @@
         <!-- Part st3215_hs_l -->
         <visual>
-        <origin xyz="0.0175 0.0452886 0.00753371" rpy="0 -0 -0"/>
+        <origin xyz="0.0175 0.0452886 0.00753371" rpy="0 0 0"/>
         <geometry>
             <mesh filename="package://gizmo_description/meshes/st3215_hs_l.stl"/>
@@ -167,5 +167,5 @@
         <!-- Part st3215_hs_r -->
         <visual>
-        <origin xyz="0.0175 -0.0452886 0.00753324" rpy="0 -0 -0"/>
+        <origin xyz="0.0175 -0.0452886 0.00753324" rpy="0 0 0"/>
         <geometry>
             <mesh filename="package://gizmo_description/meshes/st3215_hs_r.stl"/>
@@ -177,5 +177,5 @@
         <!-- Part bn_8699_1727796_hexagon_socket_button_head_screw_m2_5x6_4 -->
         <visual>
-        <origin xyz="0.001 0.0627386 0.03011" rpy="3.14159 0 -1.5708"/>
+        <origin xyz="0.001 0.0627386 0.03011" rpy="${pi} 0 -${pi/2}"/>
         <geometry>
             <mesh filename="package://gizmo_description/meshes/bn_8699_1727796_hexagon_socket_button_head_screw_m2_5x6.stl"/>
@@ -187,5 +187,5 @@
         <!-- Part bn_8699_1727796_hexagon_socket_button_head_screw_m2_5x6_5 -->
         <visual>
-        <origin xyz="0.001 0.0627386 0.00961" rpy="3.14159 0 -1.5708"/>
+        <origin xyz="0.001 0.0627386 0.00961" rpy="${pi} 0 -${pi/2}"/>
         <geometry>
             <mesh filename="package://gizmo_description/meshes/bn_8699_1727796_hexagon_socket_button_head_screw_m2_5x6.stl"/>
@@ -197,5 +197,5 @@
         <!-- Part face_plate_bottom -->
         <visual>
-        <origin xyz="0.048 -0 0.0035" rpy="0 -0 0"/>
+        <origin xyz="0.048 -0 0.0035" rpy="0 0 0"/>
         <geometry>
             <mesh filename="package://gizmo_description/meshes/face_plate_bottom.stl"/>
@@ -207,5 +207,5 @@
         <!-- Part bn_1593_1348663_hexagon_socket_button_head_screw_m3x6_7 -->
         <visual>
-        <origin xyz="0.03511 -0.0337386 0.001" rpy="-0 -1.5708 0"/>
+        <origin xyz="0.03511 -0.0337386 0.001" rpy="0 -${pi/2} 0"/>
         <geometry>
             <mesh filename="package://gizmo_description/meshes/bn_1593_1348663_hexagon_socket_button_head_screw_m3x6.stl"/>
@@ -217,5 +217,5 @@
         <!-- Part bn_8699_1727796_hexagon_socket_button_head_screw_m2_5x6_6 -->
         <visual>
-        <origin xyz="0.0217 -0.0627386 0.03011" rpy="1.5708 -0 1.5708"/>
+        <origin xyz="0.0217 -0.0627386 0.03011" rpy="${pi/2} 0 ${pi/2}"/>
         <geometry>
             <mesh filename="package://gizmo_description/meshes/bn_8699_1727796_hexagon_socket_button_head_screw_m2_5x6.stl"/>
@@ -227,5 +227,5 @@
         <!-- Part bn_1593_1348663_hexagon_socket_button_head_screw_m3x6_8 -->
         <visual>
-        <origin xyz="0.03511 -0.0557386 0.001" rpy="-0 -1.5708 0"/>
+        <origin xyz="0.03511 -0.0557386 0.001" rpy="0 -${pi/2} 0"/>
         <geometry>
             <mesh filename="package://gizmo_description/meshes/bn_1593_1348663_hexagon_socket_button_head_screw_m3x6.stl"/>
@@ -237,5 +237,5 @@
         <!-- Part bn_8699_1727796_hexagon_socket_button_head_screw_m2_5x6_7 -->
         <visual>
-        <origin xyz="0.001 -0.0627386 0.03011" rpy="1.5708 -0 1.5708"/>
+        <origin xyz="0.001 -0.0627386 0.03011" rpy="${pi/2} 0 ${pi/2}"/>
         <geometry>
             <mesh filename="package://gizmo_description/meshes/bn_8699_1727796_hexagon_socket_button_head_screw_m2_5x6.stl"/>
@@ -247,5 +247,5 @@
         <!-- Part bn_1593_1348663_hexagon_socket_button_head_screw_m3x6_9 -->
         <visual>
-        <origin xyz="-0.00011 0.0557386 0.001" rpy="-0 -1.5708 0"/>
+        <origin xyz="-0.00011 0.0557386 0.001" rpy="0 -${pi/2} 0"/>
         <geometry>
             <mesh filename="package://gizmo_description/meshes/bn_1593_1348663_hexagon_socket_button_head_screw_m3x6.stl"/>
@@ -257,5 +257,5 @@
         <!-- Part bn_8699_1727796_hexagon_socket_button_head_screw_m2_5x6_8 -->
         <visual>
-        <origin xyz="0.0217 0.0627386 0.03011" rpy="3.14159 0 -1.5708"/>
+        <origin xyz="0.0217 0.0627386 0.03011" rpy="${pi} 0 -${pi/2}"/>
         <geometry>
             <mesh filename="package://gizmo_description/meshes/bn_8699_1727796_hexagon_socket_button_head_screw_m2_5x6.stl"/>
@@ -267,5 +267,5 @@
         <!-- Part bn_1593_1348663_hexagon_socket_button_head_screw_m3x6_10 -->
         <visual>
-        <origin xyz="-0.00011 -0.0557386 0.001" rpy="-0 -1.5708 0"/>
+        <origin xyz="-0.00011 -0.0557386 0.001" rpy="0 -${pi/2} 0"/>
         <geometry>
             <mesh filename="package://gizmo_description/meshes/bn_1593_1348663_hexagon_socket_button_head_screw_m3x6.stl"/>

File: src/gizmo/gizmo_description/urdf/include/base_floor2.xacro (robot description, xacro)
@@ -17,5 +17,5 @@
         <!-- Part base_floor_2 -->
         <visual>
-        <origin xyz="0 0 0" rpy="0 -0 0"/>
+        <origin xyz="0 0 0" rpy="0 0 0"/>
         <geometry>
             <mesh filename="package://gizmo_description/meshes/base_floor_2.stl"/>
@@ -27,5 +27,5 @@
         <!-- Part bn_1593_1348663_hexagon_socket_button_head_screw_m3x6_11 -->
         <visual>
-        <origin xyz="-0.0406106 -0.0507522 0.001" rpy="-0 -1.5708 0"/>
+        <origin xyz="-0.0406106 -0.0507522 0.001" rpy="0 -${pi/2} 0"/>
         <geometry>
             <mesh filename="package://gizmo_description/meshes/bn_1593_1348663_hexagon_socket_button_head_screw_m3x6.stl"/>
@@ -37,5 +37,5 @@
         <!-- Part face_plate_top -->
         <visual>
-        <origin xyz="0.048 0 0.0035" rpy="0 -0 0"/>
+        <origin xyz="0.048 0 0.0035" rpy="0 0 0"/>
         <geometry>
             <mesh filename="package://gizmo_description/meshes/face_plate_top.stl"/>
@@ -47,5 +47,5 @@
         <!-- Part bn_1593_1348663_hexagon_socket_button_head_screw_m3x6_12 -->
         <visual>
-        <origin xyz="-0.0406106 0.0507522 0.001" rpy="-0 -1.5708 0"/>
+        <origin xyz="-0.0406106 0.0507522 0.001" rpy="0 -${pi/2} 0"/>
         <geometry>
             <mesh filename="package://gizmo_description/meshes/bn_1593_1348663_hexagon_socket_button_head_screw_m3x6.stl"/>
@@ -57,5 +57,5 @@
         <!-- Part standoff_spacer_m3_20mm -->
         <visual>
-        <origin xyz="-0.0406106 0.0507522 0.0035" rpy="0 -0 0"/>
+        <origin xyz="-0.0406106 0.0507522 0.0035" rpy="0 0 0"/>
         <geometry>
             <mesh filename="package://gizmo_description/meshes/standoff_spacer_m3_20mm.stl"/>
@@ -67,5 +67,5 @@
         <!-- Part standoff_spacer_m3_20mm_2 -->
         <visual>
-        <origin xyz="-0.0406106 -0.0507522 0.0035" rpy="0 -0 0"/>
+        <origin xyz="-0.0406106 -0.0507522 0.0035" rpy="0 0 0"/>
         <geometry>
             <mesh filename="package://gizmo_description/meshes/standoff_spacer_m3_20mm.stl"/>
@@ -77,5 +77,5 @@
         <!-- Part mcu_controller -->
         <visual>
-        <origin xyz="0 0 0.0035" rpy="0 -0 0"/>
+        <origin xyz="0 0 0.0035" rpy="0 0 0"/>
         <geometry>
             <mesh filename="package://gizmo_description/meshes/mcu_controller.stl"/>

File: src/gizmo/gizmo_description/urdf/include/base_floor3.xacro (robot description, xacro)
@@ -17,5 +17,5 @@
         <!-- Part base_floor_3 -->
         <visual>
-            <origin xyz="0 0 0" rpy="0 -0 0"/>
+            <origin xyz="0 0 0" rpy="0 0 0"/>
             <geometry>
                 <mesh filename="package://gizmo_description/meshes/base_floor_3.stl"/>
@@ -27,5 +27,5 @@
         <!-- Part bn_1593_1348663_hexagon_socket_button_head_screw_m3x6_13 -->
         <visual>
-        <origin xyz="-0.0406106 -0.0507522 0.002" rpy="-0 1.5708 0"/>
+        <origin xyz="-0.0406106 -0.0507522 0.002" rpy="0 ${pi/2} 0"/>
         <geometry>
             <mesh filename="package://gizmo_description/meshes/bn_1593_1348663_hexagon_socket_button_head_screw_m3x6.stl"/>
@@ -37,5 +37,5 @@
         <!-- Part bn_1593_1348663_hexagon_socket_button_head_screw_m3x6_14 -->
         <visual>
-        <origin xyz="-0.0406106 0.0507522 0.002" rpy="-0 1.5708 0"/>
+        <origin xyz="-0.0406106 0.0507522 0.002" rpy="0 ${pi/2} 0"/>
         <geometry>
             <mesh filename="package://gizmo_description/meshes/bn_1593_1348663_hexagon_socket_button_head_screw_m3x6.stl"/>

File: src/gizmo/gizmo_description/urdf/include/caster_wheel.xacro (robot description, xacro)
@@ -17,5 +17,5 @@
         <!-- Part caster_ball -->
         <visual>
-        <origin xyz="0 0 0" rpy="0 -0 0"/>
+        <origin xyz="0 0 0" rpy="0 0 0"/>
         <geometry>
             <mesh filename="package://gizmo_description/meshes/caster_ball.stl"/>
@@ -27,5 +27,5 @@
         <!-- Part caster_frame -->
         <visual>
-        <origin xyz="0 0 0" rpy="0 -0 0"/>
+        <origin xyz="0 0 0" rpy="0 0 0"/>
         <geometry>
             <mesh filename="package://gizmo_description/meshes/caster_frame.stl"/>

File: src/gizmo/gizmo_description/urdf/include/wheel_left.xacro (robot description, xacro)
@@ -20,5 +20,5 @@
     <!-- Part 25t_servo_horn_l -->
     <visual>
-      <origin xyz="0 -0.00699 0" rpy="0 -0 -0"/>
+      <origin xyz="0 -0.00699 0" rpy="0 0 0"/>
       <geometry>
         <mesh filename="package://gizmo_description/meshes/25t_servo_horn_l.stl"/>
@@ -30,5 +30,5 @@
     <!-- Part servo_horn_adapter_wheel70mm__l -->
     <visual>
-      <origin xyz="0 -0.0045 0" rpy="0 -0 -0"/>
+      <origin xyz="0 -0.0045 0" rpy="0 0 0"/>
       <geometry>
         <mesh filename="package://gizmo_description/meshes/servo_horn_adapter_wheel70mm__l.stl"/>
@@ -40,5 +40,5 @@
     <!-- Part rim -->
     <visual>
-      <origin xyz="0 0 0" rpy="0 -0 -0"/>
+      <origin xyz="0 0 0" rpy="0 0 0"/>
       <geometry>
         <mesh filename="package://gizmo_description/meshes/rim.stl"/>
@@ -50,5 +50,5 @@
     <!-- Part tire -->
     <visual>
-      <origin xyz="0 0 0" rpy="0 -0 -0"/>
+      <origin xyz="0 0 0" rpy="0 0 0"/>
       <geometry>
         <mesh filename="package://gizmo_description/meshes/tire.stl"/>
@@ -60,5 +60,5 @@
     <!-- Part bn_1593_1348663_hexagon_socket_button_head_screw_m3x6_15 -->
     <visual>
-      <origin xyz="-0.00824889 0.0015 -0.0047625" rpy="1.5708 0 -1.5708"/>
+      <origin xyz="-0.00824889 0.0015 -0.0047625" rpy="${pi/2} 0 -${pi/2}"/>
       <geometry>
         <mesh filename="package://gizmo_description/meshes/bn_1593_1348663_hexagon_socket_button_head_screw_m3x6.stl"/>
@@ -70,5 +70,5 @@
     <!-- Part bn_1593_1348663_hexagon_socket_button_head_screw_m3x6_16 -->
     <visual>
-      <origin xyz="0 0.0015 0.009525" rpy="1.5708 0 -1.5708"/>
+      <origin xyz="0 0.0015 0.009525" rpy="${pi/2} 0 -${pi/2}"/>
       <geometry>
         <mesh filename="package://gizmo_description/meshes/bn_1593_1348663_hexagon_socket_button_head_screw_m3x6.stl"/>
@@ -80,5 +80,5 @@
     <!-- Part bn_1593_1348663_hexagon_socket_button_head_screw_m3x6_17 -->
     <visual>
-      <origin xyz="0.00824889 0.0015 -0.0047625" rpy="1.5708 0 -1.5708"/>
+      <origin xyz="0.00824889 0.0015 -0.0047625" rpy="${pi/2} 0 -${pi/2}"/>
       <geometry>
         <mesh filename="package://gizmo_description/meshes/bn_1593_1348663_hexagon_socket_button_head_screw_m3x6.stl"/>
@@ -90,5 +90,5 @@
     <!-- Part bn_1593_1348663_hexagon_socket_button_head_screw_m3x6_18 -->
     <visual>
-      <origin xyz="0 0.0015 0" rpy="3.14159 0 -1.5708"/>
+      <origin xyz="0 0.0015 0" rpy="${pi} 0 -${pi/2}"/>
       <geometry>
         <mesh filename="package://gizmo_description/meshes/bn_1593_1348663_hexagon_socket_button_head_screw_m3x6.stl"/>

File: src/gizmo/gizmo_description/urdf/include/wheel_right.xacro (robot description, xacro)
@@ -20,5 +20,5 @@
     <!-- Part 25t_servo_horn_r -->
     <visual>
-      <origin xyz="0 0.00699 0" rpy="0 -0 0"/>
+      <origin xyz="0 0.00699 0" rpy="0 0 0"/>
       <geometry>
         <mesh filename="package://gizmo_description/meshes/25t_servo_horn_r.stl"/>
@@ -30,5 +30,5 @@
     <!-- Part servo_horn_adapter_wheel70mm__r -->
     <visual>
-      <origin xyz="0 0.0045 0" rpy="0 -0 0"/>
+      <origin xyz="0 0.0045 0" rpy="0 0 0"/>
       <geometry>
         <mesh filename="package://gizmo_description/meshes/servo_horn_adapter_wheel70mm__r.stl"/>
@@ -40,5 +40,5 @@
     <!-- Part rim_2 -->
     <visual>
-      <origin xyz="0 0 0" rpy="0 -0 0"/>
+      <origin xyz="0 0 0" rpy="0 0 0"/>
       <geometry>
         <mesh filename="package://gizmo_description/meshes/rim.stl"/>
@@ -50,5 +50,5 @@
     <!-- Part tire_2 -->
     <visual>
-      <origin xyz="0 0 0" rpy="0 -0 0"/>
+      <origin xyz="0 0 0" rpy="0 0 0"/>
       <geometry>
         <mesh filename="package://gizmo_description/meshes/tire.stl"/>
@@ -60,5 +60,5 @@
     <!-- Part bn_1593_1348663_hexagon_socket_button_head_screw_m3x6_19 -->
     <visual>
-      <origin xyz="-0.00824889 -0.0015 -0.0047625" rpy="-1.5708 -0 1.5708"/>
+      <origin xyz="-0.00824889 -0.0015 -0.0047625" rpy="-${pi/2} 0 ${pi/2}"/>
       <geometry>
         <mesh filename="package://gizmo_description/meshes/bn_1593_1348663_hexagon_socket_button_head_screw_m3x6.stl"/>
@@ -70,5 +70,5 @@
     <!-- Part bn_1593_1348663_hexagon_socket_button_head_screw_m3x6_20 -->
     <visual>
-      <origin xyz="0 -0.0015 0.009525" rpy="-1.5708 -0 1.5708"/>
+      <origin xyz="0 -0.0015 0.009525" rpy="-${pi/2} 0 ${pi/2}"/>
       <geometry>
         <mesh filename="package://gizmo_description/meshes/bn_1593_1348663_hexagon_socket_button_head_screw_m3x6.stl"/>
@@ -80,5 +80,5 @@
     <!-- Part bn_1593_1348663_hexagon_socket_button_head_screw_m3x6_21 -->
     <visual>
-      <origin xyz="0 -0.0015 0" rpy="-1.5708 -0 1.5708"/>
+      <origin xyz="0 -0.0015 0" rpy="-${pi/2} 0 ${pi/2}"/>
       <geometry>
         <mesh filename="package://gizmo_description/meshes/bn_1593_1348663_hexagon_socket_button_head_screw_m3x6.stl"/>
@@ -90,5 +90,5 @@
     <!-- Part bn_1593_1348663_hexagon_socket_button_head_screw_m3x6_22 -->
     <visual>
-      <origin xyz="0.00824889 -0.0015 -0.0047625" rpy="-1.5708 -0 1.5708"/>
+      <origin xyz="0.00824889 -0.0015 -0.0047625" rpy="-${pi/2} 0 ${pi/2}"/>
       <geometry>
         <mesh filename="package://gizmo_description/meshes/bn_1593_1348663_hexagon_socket_button_head_screw_m3x6.stl"/>
