Commit message: feat: standardize joint naming in robot description

File: src/gizmo/gizmo_description/urdf/include/gizmo_mobile_base.xacro (robot description, xacro)
@@ -17,5 +17,5 @@
     <link name="base_footprint"/>
     <!-- Joint base_footprint_base_floor1 -->
-    <joint name="base_footprint_base_floor1" type="fixed">
+    <joint name="base_footprint_joint" type="fixed">
         <origin xyz="${base_footprint_base_floor1_o_xyz}" rpy="0 0 0"/>
         <parent link="base_footprint"/>
@@ -23,5 +23,5 @@
     </joint>
     <!-- Joint base_floor1_base_floor2 -->
-    <joint name="base_floor1_base_floor2" type="fixed">
+    <joint name="base_floor1_base_floor2_joint" type="fixed">
         <origin xyz="${base_floor1_base_floor2_o_xyz}" rpy="0 0 0"/>
         <parent link="base_floor1"/>
@@ -29,5 +29,5 @@
     </joint>
     <!-- Joint base_floor2_base_floor3 -->
-    <joint name="base_floor2_base_floor3" type="fixed">
+    <joint name="base_floor2_base_floor3_joint" type="fixed">
         <origin xyz="${base_floor2_base_floor3_o_xyz}" rpy="0 0 0"/>
         <parent link="base_floor2"/>
@@ -35,5 +35,5 @@
     </joint>
     <!-- Joint base_floor1_caster_wheel -->
-    <joint name="base_floor1_caster_wheel" type="fixed">
+    <joint name="caster_wheel_joint" type="fixed">
         <origin xyz="${base_floor1_caster_wheel_o_xyz}" rpy="0 0 0"/>
         <parent link="base_floor1"/>
@@ -41,5 +41,5 @@
     </joint>
     <!-- Joint base_floor1_wheel_left -->
-    <joint name="base_floor1_wheel_left" type="continuous">
+    <joint name="left_wheel_joint" type="continuous">
         <origin xyz="${base_floor1_wheel_left_o_xyz}" rpy="0 0 0"/>
         <parent link="base_floor1"/>
@@ -49,5 +49,5 @@
     </joint>
     <!-- Joint base_floor1_wheel_right -->
-    <joint name="base_floor1_wheel_right" type="continuous">
+    <joint name="right_wheel_joint" type="continuous">
         <origin xyz="${base_floor1_wheel_right_o_xyz}" rpy="0 0 0"/>
         <parent link="base_floor1"/>

Commit message: fix(gizmo_description): resolve velocity blending failure during curved turns
- Remove artificial 10 rad/s velocity limits on left_wheel_joint and right_wheel_joint
- Fix issue where combined cmd_vel (linear + angular) prioritized straight line driving over curve turning due to wheel speed saturation
- Enable smooth differential curve blending in Gazebo Sim

File: src/gizmo/gizmo_description/urdf/include/gizmo_mobile_base.xacro (robot description, xacro)
@@ -46,5 +46,5 @@
         <child link="wheel_left"/>
         <axis xyz="0 1 0"/>
-        <limit effort="10" velocity="10"/>
+        <!-- <limit effort="10" velocity="10"/> -->
     </joint>
     <!-- Joint base_floor1_wheel_right -->
@@ -54,5 +54,5 @@
         <child link="wheel_right"/>
         <axis xyz="0 1 0"/>
-        <limit effort="10" velocity="10"/>
+        <!-- <limit effort="10" velocity="10"/> -->
     </joint>
 </robot>
