Commit message: fix: update Gazebo diff_drive plugin acceleration limits and wheel friction parameters

File: src/gizmo/gizmo_description/robot.urdf (robot description, URDF)
Before this commit: robot gizmo, 9 links, 8 joints
Links:
- removed link bno055
- removed link lidar
- removed link realsense_d435
- added link base_footprint
- link base_floor1: geometry collision cylinder length=0.0335 radius=0.075; visual mesh filename=package://gizmo_description/meshes/base_floor_1.stl
- link base_floor2: geometry collision cylinder length=0.0235 radius=0.075; visual mesh filename=package://gizmo_description/meshes/base_floor_2.stl
- link base_floor3: geometry collision cylinder length=0.003 radius=0.075; visual mesh filename=package://gizmo_description/meshes/base_floor_3.stl
- link caster_wheel: geometry collision sphere radius=0.00756558; visual mesh filename=package://gizmo_description/meshes/caster_ball.stl
- link wheel_left: geometry collision sphere radius=0.035; visual mesh filename=package://gizmo_description/meshes/25t_servo_horn_l.stl
- link wheel_right: geometry collision sphere radius=0.035; visual mesh filename=package://gizmo_description/meshes/25t_servo_horn_r.stl
Joints:
- removed joint base_Floor2_joint
- removed joint base_Floor3_joint
- removed joint camera_joint
- removed joint caster_joint
- removed joint imu_joint
- removed joint lidar_joint
- added joint base_floor1_base_floor2_joint: type fixed, parent base_floor1, child base_floor2, origin xyz=0 0 0.03350000 rpy=0 0 0
- added joint base_floor2_base_floor3_joint: type fixed, parent base_floor2, child base_floor3, origin xyz=0 0 0.02350000 rpy=0 0 0
- added joint base_footprint_joint: type fixed, parent base_footprint, child base_floor1, origin xyz=0 0 0.01163116 rpy=0 0 0
- added joint caster_wheel_joint: type fixed, parent base_floor1, child caster_wheel, origin xyz=-0.0556106 -0 0.0035 rpy=0 0 0
- joint left_wheel_joint: axis 0 0 1 -> 0 1 0; origin xyz=0.03 0.0601386 0.01986 rpy=-0 0 -0 -> xyz=0.03 0.0691386 0.01986 rpy=0 0 0
- joint right_wheel_joint: axis 0 0 1 -> 0 1 0; origin xyz=0.03 -0.0601386 0.01986 rpy=0 -0 -0 -> xyz=0.03 -0.0691386 0.01986 rpy=0 0 0

File: src/gizmo/gizmo_description/urdf/include/gizmo_mobile_base.gazebo.xacro (robot description, xacro)
@@ -5,6 +5,6 @@
     <!-- Left Wheel Surface Friction & Contact Stability -->
     <gazebo reference="wheel_left">
-        <mu1>1.0</mu1>
-        <mu2>1.0</mu2>
+        <mu1>1000000000000000.0</mu1>
+        <mu2>1000000000000000.0</mu2>
         <kp>1000000000000.0</kp>
         <kd>10.0</kd>
@@ -15,6 +15,6 @@
     <!-- Right Wheel Surface Friction & Contact Stability -->
     <gazebo reference="wheel_right">
-        <mu1>1.0</mu1>
-        <mu2>1.0</mu2>
+        <mu1>1000000000000000.0</mu1>
+        <mu2>1000000000000000.0</mu2>
         <kp>1000000000000.0</kp>
         <kd>10.0</kd>
@@ -42,9 +42,9 @@
             <wheel_radius>${wheel_radius}</wheel_radius>
             <!-- Limits & Acceleration -->
-            <max_linear_acceleration>1.0</max_linear_acceleration>
-            <min_linear_acceleration>-1.0</min_linear_acceleration>
-            <max_angular_acceleration>2.0</max_angular_acceleration>
-            <min_angular_acceleration>-2.0</min_angular_acceleration>
-            <max_torque>10.0</max_torque>
+            <max_linear_acceleration>10.0</max_linear_acceleration>
+            <min_linear_acceleration>-10.0</min_linear_acceleration>
+            <max_angular_acceleration>20.0</max_angular_acceleration>
+            <min_angular_acceleration>-20.0</min_angular_acceleration>
+            <max_torque>50.0</max_torque>
             <!-- Topics & Frames -->
             <topic>/cmd_vel</topic>

Commit message: ...

File: src/gizmo/gizmo_description/robot.urdf (robot description, URDF)
Before this commit: robot gizmo, 7 links, 6 joints
Links:
- removed link base_footprint
- added link bno055, mass 0.003; collision mesh filename=package://gizmo_description/meshes/bno055.stl; visual mesh filename=package://gizmo_description/meshes/bno055.stl
- added link lidar, mass 0.19; collision mesh filename=package://gizmo_description/meshes/lidar.stl; visual mesh filename=package://gizmo_description/meshes/lidar.stl
- added link realsense_d435, mass 0.049866; collision mesh filename=package://gizmo_description/meshes/realsense_d435.stl; visual mesh filename=package://gizmo_description/meshes/realsense_d435.stl
- link base_floor1: geometry collision mesh filename=package://gizmo_description/meshes/base_floor_1.stl; collision mesh filename=package://gizmo_description/meshes/bn_1593_1348663_hexagon_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
- link base_floor2: geometry collision mesh filename=package://gizmo_description/meshes/base_floor_2.stl; collision mesh filename=package://gizmo_description/meshes/bn_1593_1348663_hexagon_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
- link base_floor3: geometry collision mesh filename=package://gizmo_description/meshes/base_floor_3.stl; collision mesh filename=package://gizmo_description/meshes/bn_1593_1348663_hexagon_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
- link caster_wheel: geometry collision mesh filename=package://gizmo_description/meshes/caster_ball.stl; collision mesh filename=package://gizmo_description/meshes/caster_frame.stl
- link wheel_left: geometry collision mesh filename=package://gizmo_description/meshes/25t_servo_horn_l.stl; collision mesh filename=package://gizmo_description/meshes/bn_1593_1348663_hexagon_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
- link wheel_right: geometry collision mesh filename=package://gizmo_description/meshes/25t_servo_horn_r.stl; collision mesh filename=package://gizmo_description/meshes/bn_1593_1348663_hexagon_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
Joints:
- removed joint base_floor1_base_floor2_joint
- removed joint base_floor2_base_floor3_joint
- removed joint base_footprint_joint
- removed joint caster_wheel_joint
- added joint base_Floor2_joint: type fixed, parent base_floor1, child base_floor2, origin xyz=0 0 0.0335 rpy=0 -0 0, axis 0 0 1, limit effort=10 velocity=10
- added joint base_Floor3_joint: type fixed, parent base_floor2, child base_floor3, origin xyz=0 0 0.0235 rpy=0 -0 0, axis 0 0 1, limit effort=10 velocity=10
- added joint camera_joint: type fixed, parent base_floor3, child realsense_d435, origin xyz=0.055 -0 0.003 rpy=0 -0 0, axis 0 0 1, limit effort=10 velocity=10
- added joint caster_joint: type fixed, parent base_floor1, child caster_wheel, origin xyz=-0.0556106 -0 0.0035 rpy=0 -0 0, axis 0 0 1, limit effort=10 velocity=10
- added joint imu_joint: type fixed, parent base_floor1, child bno055, origin xyz=0 0 0.0035 rpy=0 -0 0, axis 0 0 1, limit effort=10 velocity=10
- added joint lidar_joint: type fixed, parent base_floor3, child lidar, origin xyz=0 0 0.003 rpy=0 -0 0, axis 0 0 1, limit effort=10 velocity=10
- joint left_wheel_joint: axis 0 1 0 -> 0 0 1; origin xyz=0.03 0.0691386 0.01986 rpy=0 0 0 -> xyz=0.03 0.0601386 0.01986 rpy=-0 0 -0
- joint right_wheel_joint: axis 0 1 0 -> 0 0 1; origin xyz=0.03 -0.0691386 0.01986 rpy=0 0 0 -> xyz=0.03 -0.0601386 0.01986 rpy=0 -0 -0

Commit message: refactor(gizmo_description): update caster wheel height, mass, and inertia properties
- Correct caster wheel height dimension in CAD model to level the robot base
- Update caster link mass and inertia tensor calculations accordingly
- Fix slight chassis pitch tilt, aligning base_footprint and LiDAR scan plane perfectly horizontal to ground

File: src/gizmo/gizmo_description/robot.urdf (robot description, URDF)
Before this commit: robot gizmo, 9 links, 8 joints
Links:
- link caster_wheel: mass 0.00663696 -> 0.00740259

File: src/gizmo/gizmo_description/urdf/include/caster_wheel.xacro (robot description, xacro)
@@ -1,6 +1,6 @@
 <?xml version="1.0" ?>
 <robot xmlns:xacro="http://www.ros.org/wiki/xacro">
-    <xacro:property name="caster_wheel_m" value="0.00663696" />
-    <xacro:property name="caster_wheel_d" value="0.01513116" />
+    <xacro:property name="caster_wheel_m" value="0.00740259" />
+    <xacro:property name="caster_wheel_d" value="0.01863116" />
     <xacro:property name="caster_wheel_r" value="${caster_wheel_d / 2}" />
     <xacro:property name="caster_wheel_o_xyz" value="0 0 -${caster_wheel_r}" />

File: src/gizmo/gizmo_description/urdf/include/gizmo_mobile_base.xacro (robot description, xacro)
@@ -8,5 +8,5 @@
     <xacro:include filename="$(find gizmo_description)/urdf/include/wheel_left.xacro" />
     <xacro:include filename="$(find gizmo_description)/urdf/include/wheel_right.xacro" />
-    <xacro:property name="base_footprint_base_floor1_o_xyz" value="0 0 0.01163116" />
+    <xacro:property name="base_footprint_base_floor1_o_xyz" value="0 0 0.01513116" />
     <xacro:property name="base_floor1_base_floor2_o_xyz" value="0 0 0.03350000" />
     <xacro:property name="base_floor2_base_floor3_o_xyz" value="0 0 0.02350000" />
