Commit message: refactor: rename lidar link and associated joint to lidar_link for consistency

File: src/gizmo/gizmo_description/urdf/include/robot_components/lidar.xacro (robot description, xacro)
@@ -6,6 +6,6 @@
     <xacro:property name="lidar_o_xyz" value="0 0 ${lidar_length/2}" />
     <xacro:property name="lidar_o_rpy" value="0 0 0" />
-    <!-- Link lidar -->
-    <link name="lidar">
+    <!-- Link lidar_link -->
+    <link name="lidar_link">
         <xacro:cylinder_inertia m="${lidar_m}" r="${lidar_r}" h="${lidar_length}" o_xyz="${lidar_o_xyz}" o_rpy="${lidar_o_rpy}"/>
         <collision>

File: src/gizmo/gizmo_description/urdf/include/robot_components/sensors.xacro (robot description, xacro)
@@ -5,6 +5,6 @@
     <xacro:include filename="$(find gizmo_description)/urdf/include/robot_components/camera.xacro" />
     <!-- lidar properties -->
-    <xacro:property name="base_floor3_lidar_o_xyz" value="0 0 0.003" />
-    <xacro:property name="base_floor3_lidar_o_rpy" value="0 0 0" />
+    <xacro:property name="base_floor3_lidar_link_o_xyz" value="0 0 0.003" />
+    <xacro:property name="base_floor3_lidar_link_o_rpy" value="0 0 0" />
     <xacro:property name="lidar_scan_frame_o_xyz" value="0 0 0.031" />
     <xacro:property name="lidar_scan_frame_o_rpy" value="0 0 0" />
@@ -14,13 +14,13 @@
     <xacro:property name="camera_optical_frame_o_xyz" value="0.01342258 0 0.01237412" />
     <xacro:property name="camera_optical_frame_o_rpy" value="${-pi/2} 0 ${-pi/2}" />
-    <!-- Joint lidar -->
-    <joint name="lidar_joint" type="fixed">
-        <origin xyz="${base_floor3_lidar_o_xyz}" rpy="${base_floor3_lidar_o_rpy}"/>
+    <!-- Joint lidar_link -->
+    <joint name="lidar_link_joint" type="fixed">
+        <origin xyz="${base_floor3_lidar_link_o_xyz}" rpy="${base_floor3_lidar_link_o_rpy}"/>
         <parent link="base_floor3"/>
-        <child link="lidar"/>
+        <child link="lidar_link"/>
     </joint>
     <joint name="scan_frame_joint" type="fixed">
         <origin xyz="${lidar_scan_frame_o_xyz}" rpy="${lidar_scan_frame_o_rpy}"/>
-        <parent link="lidar"/>
+        <parent link="lidar_link"/>
         <child link="scan_frame"/>
     </joint>
