Commit message: fix(urdf): reorder visual elements for correct link color rendering in RViz2
RViz2's RobotLink implementation (rviz_default_plugins) retrieves the default
link material from the link's first <visual> element and assigns it to all
STL meshes attached to that link (since STL files lack embedded material data).

Previously, base_floor1, caster_wheel, wheel_left, and wheel_right declared
screws or ball bearings with light silver/grey materials as their first visual,
causing RViz2 to tint the entire chassis floor, caster assembly, and wheels grey.

This change places each link's primary body mesh first:
- base_floor1: base_floor_1 (dark charcoal/black)
- caster_wheel: caster_frame (teal)
- wheel_left: rim (teal) and tire (dark charcoal)
- wheel_right: rim_2 (teal) and tire_2 (dark charcoal)

This guarantees RViz2 renders the robot links in their intended colors without
altering physical joints, inertia, or collision geometry.

File: src/gizmo/gizmo_description/urdf/include/robot_components/base_floor1.xacro (robot description, xacro)
@@ -15,4 +15,14 @@
         </geometry>
         </collision>
+        <!-- Part base_floor_1 -->
+        <visual>
+        <origin xyz="0 0 0" rpy="0 0 0"/>
+        <geometry>
+            <mesh filename="package://gizmo_description/meshes/base_floor_1.stl"/>
+        </geometry>
+        <material name="base_floor_1_material">
+            <color rgba="0.121569 0.133333 0.14902 1"/>
+        </material>
+        </visual>
         <!-- Part bn_8699_1727796_hexagon_socket_button_head_screw_m2_5x6 -->
         <visual>
@@ -105,14 +115,4 @@
         </material>
         </visual>
-        <!-- Part base_floor_1 -->
-        <visual>
-        <origin xyz="0 0 0" rpy="0 0 0"/>
-        <geometry>
-            <mesh filename="package://gizmo_description/meshes/base_floor_1.stl"/>
-        </geometry>
-        <material name="base_floor_1_material">
-            <color rgba="0.121569 0.133333 0.14902 1"/>
-        </material>
-        </visual>
         <!-- Part servo_bracket_r -->
         <visual>

File: src/gizmo/gizmo_description/urdf/include/robot_components/caster_wheel.xacro (robot description, xacro)
@@ -15,4 +15,14 @@
             </geometry>
         </collision>
+        <!-- Part caster_frame -->
+        <visual>
+        <origin xyz="0 0 0" rpy="0 0 0"/>
+        <geometry>
+            <mesh filename="package://gizmo_description/meshes/caster_frame.stl"/>
+        </geometry>
+        <material name="caster_frame_material">
+            <color rgba="0.141176 0.694118 0.65098 1"/>
+        </material>
+        </visual>
         <!-- Part caster_ball -->
         <visual>
@@ -25,14 +35,4 @@
         </material>
         </visual>
-        <!-- Part caster_frame -->
-        <visual>
-        <origin xyz="0 0 0" rpy="0 0 0"/>
-        <geometry>
-            <mesh filename="package://gizmo_description/meshes/caster_frame.stl"/>
-        </geometry>
-        <material name="caster_frame_material">
-            <color rgba="0.141176 0.694118 0.65098 1"/>
-        </material>
-        </visual>
     </link>
 </robot>

File: src/gizmo/gizmo_description/urdf/include/robot_components/wheel_left.xacro (robot description, xacro)
@@ -18,4 +18,24 @@
       </geometry>
     </collision>
+    <!-- Part rim -->
+    <visual>
+      <origin xyz="0 0 0" rpy="0 0 0"/>
+      <geometry>
+        <mesh filename="package://gizmo_description/meshes/rim.stl"/>
+      </geometry>
+      <material name="rim_material">
+        <color rgba="0.0941176 0.580392 0.545098 1"/>
+      </material>
+    </visual>
+    <!-- Part tire -->
+    <visual>
+      <origin xyz="0 0 0" rpy="0 0 0"/>
+      <geometry>
+        <mesh filename="package://gizmo_description/meshes/tire.stl"/>
+      </geometry>
+      <material name="tire_material">
+        <color rgba="0.0784314 0.0784314 0.0784314 1"/>
+      </material>
+    </visual>
     <!-- Part 25t_servo_horn_l -->
     <visual>
@@ -36,24 +56,4 @@
       <material name="servo_horn_adapter_wheel70mm__l_material">
         <color rgba="0.615686 0.811765 0.929412 1"/>
-      </material>
-    </visual>
-    <!-- Part rim -->
-    <visual>
-      <origin xyz="0 0 0" rpy="0 0 0"/>
-      <geometry>
-        <mesh filename="package://gizmo_description/meshes/rim.stl"/>
-      </geometry>
-      <material name="rim_material">
-        <color rgba="0.0941176 0.580392 0.545098 1"/>
-      </material>
-    </visual>
-    <!-- Part tire -->
-    <visual>
-      <origin xyz="0 0 0" rpy="0 0 0"/>
-      <geometry>
-        <mesh filename="package://gizmo_description/meshes/tire.stl"/>
-      </geometry>
-      <material name="tire_material">
-        <color rgba="0.0784314 0.0784314 0.0784314 1"/>
       </material>
     </visual>

File: src/gizmo/gizmo_description/urdf/include/robot_components/wheel_right.xacro (robot description, xacro)
@@ -18,4 +18,24 @@
       </geometry>
     </collision>
+    <!-- Part rim_2 -->
+    <visual>
+      <origin xyz="0 0 0" rpy="0 0 0"/>
+      <geometry>
+        <mesh filename="package://gizmo_description/meshes/rim.stl"/>
+      </geometry>
+      <material name="rim_2_material">
+        <color rgba="0.0941176 0.580392 0.545098 1"/>
+      </material>
+    </visual>
+    <!-- Part tire_2 -->
+    <visual>
+      <origin xyz="0 0 0" rpy="0 0 0"/>
+      <geometry>
+        <mesh filename="package://gizmo_description/meshes/tire.stl"/>
+      </geometry>
+      <material name="tire_2_material">
+        <color rgba="0.0784314 0.0784314 0.0784314 1"/>
+      </material>
+    </visual>
     <!-- Part 25t_servo_horn_r -->
     <visual>
@@ -36,24 +56,4 @@
       <material name="servo_horn_adapter_wheel70mm__r_material">
         <color rgba="0.615686 0.811765 0.929412 1"/>
-      </material>
-    </visual>
-    <!-- Part rim_2 -->
-    <visual>
-      <origin xyz="0 0 0" rpy="0 0 0"/>
-      <geometry>
-        <mesh filename="package://gizmo_description/meshes/rim.stl"/>
-      </geometry>
-      <material name="rim_2_material">
-        <color rgba="0.0941176 0.580392 0.545098 1"/>
-      </material>
-    </visual>
-    <!-- Part tire_2 -->
-    <visual>
-      <origin xyz="0 0 0" rpy="0 0 0"/>
-      <geometry>
-        <mesh filename="package://gizmo_description/meshes/tire.stl"/>
-      </geometry>
-      <material name="tire_2_material">
-        <color rgba="0.0784314 0.0784314 0.0784314 1"/>
       </material>
     </visual>
