Commit message: fix(wheel_right): correct xacro syntax for wheel height property

File: src/gizmo/gizmo_description/urdf/include/robot_components/wheel_right.xacro (robot description, xacro)
@@ -4,5 +4,5 @@
     <xacro:property name="wheel_right_set_o_xyz" value="0 0.0025 0" />
     <xacro:property name="wheel_right_set_o_rpy" value="${pi/2} 0 0" />
-    xacro:<xacro:property name="wheel_right_set_h" value="0.0130" />
+    <xacro:property name="wheel_right_set_h" value="0.0130" />
     <xacro:property name="wheel_right_d" value="0.070" />
     <xacro:property name="wheel_right_r" value="${wheel_right_d / 2}" />
