Commit message: feat(gizmo_description): support camera_type launch argument to switch between 2D and depth camera modes
Allow switching Gazebo camera plugin mode dynamically between standard 2D RGB ('camera') and 3D RGB-D ('depth_camera') via launch CLI argument.

File: src/gizmo/gizmo_description/urdf/include/gazebo_components/camera.gazebo.xacro (robot description, xacro)
@@ -1,9 +1,17 @@
 <?xml version="1.0" ?>
 <robot xmlns:xacro="http://www.ros.org/wiki/xacro">
+    <!-- Camera Sensor Mode Argument ('camera' or 'depth_camera') -->
+    <xacro:arg name="camera_type" default="camera"/>
+    <xacro:property name="camera_type" value="$(arg camera_type)" />
     <!-- Camera Gazebo Plugin -->
     <gazebo reference="camera_link">
-        <sensor name="camera" type="camera">
+        <sensor name="camera" type="${camera_type}">
             <pose>${camera_optical_frame_o_xyz} 0 0 0</pose>
-            <topic>camera/image_raw</topic>
+            <xacro:if value="${camera_type == 'depth_camera'}">
+                <topic>camera/depth/image_raw</topic>
+            </xacro:if>
+            <xacro:unless value="${camera_type == 'depth_camera'}">
+                <topic>camera/image_raw</topic>
+            </xacro:unless>
             <camera_info_topic>camera/camera_info</camera_info_topic>
             <gz_frame_id>camera_optical_frame</gz_frame_id>
@@ -28,4 +36,13 @@
                     <stddev>0.007</stddev>
                 </noise>
+                <xacro:if value="${camera_type == 'depth_camera'}">
+                    <depth_camera>
+                        <output>depths</output>
+                        <clip>
+                            <near>0.105</near>
+                            <far>10.0</far>
+                        </clip>
+                    </depth_camera>
+                </xacro:if>
             </camera>
         </sensor>
