Commit message: feat(gizmo_description): add RealSense D435 camera link, optical frame, and Gazebo plugin
- Add camera_link and camera_optical_frame URDF links and joints with REP-103 standard orientation
- Add Gazebo camera sensor plugin attached to camera_link with pose offset at lens center
- Configure camera_info_topic and gz_frame_id for ROS 2 Gazebo Harmonic integration
- Add /camera/image_raw and /camera/camera_info topic bridge definitions to ros_gz_bridge_config.yaml

File: src/gizmo/gizmo_description/urdf/include/gazebo_components/sensors.gazebo.xacro (robot description, xacro)
@@ -9,3 +9,5 @@
     <!-- lidar plugin -->
     <xacro:include filename="$(find gizmo_description)/urdf/include/gazebo_components/lidar.gazebo.xacro" />
+    <!-- camera plugin -->
+    <xacro:include filename="$(find gizmo_description)/urdf/include/gazebo_components/camera.gazebo.xacro" />
 </robot>

File: src/gizmo/gizmo_description/urdf/include/robot_components/sensors.xacro (robot description, xacro)
@@ -3,4 +3,5 @@
     <xacro:include filename="$(find gizmo_description)/urdf/include/robot_components/inertial_function_macros.xacro" />
     <xacro:include filename="$(find gizmo_description)/urdf/include/robot_components/lidar.xacro" />
+    <xacro:include filename="$(find gizmo_description)/urdf/include/robot_components/camera.xacro" />
     <!-- lidar properties -->
     <xacro:property name="base_floor3_lidar_o_xyz" value="0 0 0.003" />
@@ -8,4 +9,9 @@
     <xacro:property name="lidar_scan_frame_o_xyz" value="0 0 0.031" />
     <xacro:property name="lidar_scan_frame_o_rpy" value="0 0 0" />
+    <!-- camera properties -->
+    <xacro:property name="base_floor3_camera_link_o_xyz" value="0.055 0 0.003" />
+    <xacro:property name="base_floor3_camera_link_o_rpy" value="0 0 0" />
+    <xacro:property name="camera_optical_frame_o_xyz" value="0.01342258 0 0.01237412" />
+    <xacro:property name="camera_optical_frame_o_rpy" value="${-pi/2} 0 ${-pi/2}" />
     <!-- Joint lidar -->
     <joint name="lidar_joint" type="fixed">
@@ -19,3 +25,14 @@
         <child link="scan_frame"/>
     </joint>
+    <!-- Joint camera_link -->
+    <joint name="camera_link_joint" type="fixed">
+        <origin xyz="${base_floor3_camera_link_o_xyz}" rpy="${base_floor3_camera_link_o_rpy}"/>
+        <parent link="base_floor3"/>
+        <child link="camera_link"/>
+    </joint>
+    <joint name="camera_optical_frame_joint" type="fixed">
+        <origin xyz="${camera_optical_frame_o_xyz}" rpy="${camera_optical_frame_o_rpy}"/>
+        <parent link="camera_link"/>
+        <child link="camera_optical_frame"/>
+    </joint>
 </robot>

Commit message: feat(gizmo_description): add BNO055 IMU link, gazebo sensor plugin, and ROS 2 topic bridge
- Add imu_link component in imu.xacro with exact CAD dimensions (26.67mm x 20.32mm x 4.15mm) and inertia
- Mount imu_link onto base_floor1 at (0, 0, 0.0035) in sensors.xacro
- Add Gazebo Harmonic IMU sensor plugin in imu.gazebo.xacro using gz-sim-imu-system at 100 Hz
- Configure realistic Gaussian noise models for angular velocity and linear acceleration
- Add /imu/data topic bridge mapping in ros_gz_bridge_config.yaml

File: src/gizmo/gizmo_description/urdf/include/gazebo_components/sensors.gazebo.xacro (robot description, xacro)
@@ -11,3 +11,5 @@
     <!-- camera plugin -->
     <xacro:include filename="$(find gizmo_description)/urdf/include/gazebo_components/camera.gazebo.xacro" />
+    <!-- imu plugin -->
+    <xacro:include filename="$(find gizmo_description)/urdf/include/gazebo_components/imu.gazebo.xacro" />
 </robot>

File: src/gizmo/gizmo_description/urdf/include/robot_components/sensors.xacro (robot description, xacro)
@@ -4,4 +4,5 @@
     <xacro:include filename="$(find gizmo_description)/urdf/include/robot_components/lidar.xacro" />
     <xacro:include filename="$(find gizmo_description)/urdf/include/robot_components/camera.xacro" />
+    <xacro:include filename="$(find gizmo_description)/urdf/include/robot_components/imu.xacro" />
     <!-- lidar properties -->
     <xacro:property name="base_floor3_lidar_link_o_xyz" value="0 0 0.003" />
@@ -14,4 +15,7 @@
     <xacro:property name="camera_optical_frame_o_xyz" value="0.01342258 0 0.01237412" />
     <xacro:property name="camera_optical_frame_o_rpy" value="${-pi/2} 0 ${-pi/2}" />
+    <!-- imu properties -->
+    <xacro:property name="base_floor1_imu_link_o_xyz" value="0 0 0.0035" />
+    <xacro:property name="base_floor1_imu_link_o_rpy" value="0 0 0" />
     <!-- Joint lidar_link -->
     <joint name="lidar_link_joint" type="fixed">
@@ -36,3 +40,9 @@
         <child link="camera_optical_frame"/>
     </joint>
+    <!-- Joint imu_link -->
+    <joint name="imu_link_joint" type="fixed">
+        <origin xyz="${base_floor1_imu_link_o_xyz}" rpy="${base_floor1_imu_link_o_rpy}"/>
+        <parent link="base_floor1"/>
+        <child link="imu_link"/>
+    </joint>
 </robot>
